Commit message: completed URDF model according to spec and tested using rviz.launch

File: my_rb1_description/urdf/my_rb1_robot.urdf (robot description, URDF)
Before this commit: robot my_rb1_robot, 3 links, 2 joints
Links:
- added link back_caster, mass 0.0276; collision sphere radius=0.025; visual sphere radius=0.025
- added link front_caster, mass 0.0276; collision sphere radius=0.025; visual sphere radius=0.025
- added link front_laser, mass 0.0579; collision cylinder length=0.07 radius=0.025; visual cylinder length=0.07 radius=0.025
- added link left_wheel, mass 0.0331; collision cylinder length=0.04 radius=0.025; visual cylinder length=0.04 radius=0.025
- link right_wheel: geometry collision cylinder length=0.04 radius=0.025; visual cylinder length=0.04 radius=0.025
Joints:
- added joint joint_back_caster_base_footprint: type fixed, parent base_footprint, child back_caster, origin xyz=-0.1 0.0 0.015 rpy=0 0 0
- added joint joint_front_caster_base_footprint: type fixed, parent base_footprint, child front_caster, origin xyz=0.1 0.0 0.015 rpy=0 0 0
- added joint joint_front_laser_base_link: type fixed, parent base_link, child front_laser, origin xyz=0.25 0.0 0.075 rpy=0 0 0
- added joint joint_left_wheel_base_footprint: type continuous, parent base_footprint, child left_wheel, origin xyz=0.0 0.20 0.015 rpy=0 0 0, axis 0 1 0, limit effort=10000 velocity=1000
- joint joint_right_wheel_base_footprint: origin xyz=0.0 -0.20 0.01 rpy=0 0 0 -> xyz=0.0 -0.20 0.015 rpy=0 0 0

Commit message: fixed visualization with missing URDF parameter and removing joint_state_publisher_gui from gazebo launch file, as well as fixing URDF parameters to reference footprint instead of base_link

File: my_rb1_description/urdf/my_rb1_robot.urdf (robot description, URDF)
Before this commit: robot my_rb1_robot, 7 links, 6 joints
Joints:
- joint joint_back_caster_base_footprint: origin xyz=-0.1 0.0 0.015 rpy=0 0 0 -> xyz=-0.1 0.0 -0.015 rpy=0 0 0
- joint joint_front_caster_base_footprint: origin xyz=0.1 0.0 0.015 rpy=0 0 0 -> xyz=0.1 0.0 -0.015 rpy=0 0 0
- joint joint_left_wheel_base_footprint: origin xyz=0.0 0.20 0.015 rpy=0 0 0 -> xyz=0.0 0.20 -0.015 rpy=0 0 0
- joint joint_right_wheel_base_footprint: origin xyz=0.0 -0.20 0.015 rpy=0 0 0 -> xyz=0.0 -0.20 -0.015 rpy=0 0 0

Commit message: implemented feedback from Alberto (instructor) in mass properties to try to fix turning issue (but now it veers left instead of right)

File: my_rb1_description/urdf/my_rb1_robot.urdf (robot description, URDF)
Before this commit: robot my_rb1_robot, 7 links, 6 joints
Links:
- link back_caster: mass 0.0276 -> 1
- link base_link: mass 24.8207 -> 19.5
- link front_caster: mass 0.0276 -> 1
- link front_laser: mass 0.0579 -> 0.5
- link left_wheel: mass 0.0331 -> 1.5
- link right_wheel: mass 0.0331 -> 1.5
